Commit message: implemented all the qcar cameras

File: qcar_description/urdf/qcar.gazebo.xacro (robot description, xacro)
@@ -8,5 +8,5 @@
         image won't be aligned properly with the frame it is supposedly
         originating from -->
-    <origin xyz="0.01 0 0" rpy="${-pi/2} 0 ${-pi/2}"/>
+    <origin xyz="0 0 0" rpy="${-pi/2} 0 ${-pi/2}"/>
     <parent link="camera_rgb"/>
     <child link="camera_rgb_optical_link"/>
@@ -48,4 +48,205 @@
     </sensor>
   </gazebo>
+  <link name="camera_csi_front_optical_link"/>
+  <joint name="camera_csi_front_optical_joint" type="fixed">
+    <!-- these values have to be these values otherwise the gazebo camera
+        image won't be aligned properly with the frame it is supposedly
+        originating from -->
+    <origin xyz="0 0 0" rpy="${-pi/2} 0 ${-pi/2}"/>
+    <parent link="camera_csi_front"/>
+    <child link="camera_csi_front_optical_link"/>
+  </joint>
+<!-- Define all the computer vision sernsor properties -->
+	<gazebo reference="camera_csi_front">
+    <!-- <material>Gazebo/Green</material> -->
+    <sensor type="camera" name="csi_front">
+      <always_on>1</always_on>
+      <update_rate>60.0</update_rate>
+      <visualize>true</visualize>
+      <topic>qcar/csi_front/image_raw</topic>
+      <camera name="front">
+        <horizontal_fov>2.79253</horizontal_fov>
+        <image>
+            <width>1280</width>
+            <height>640</height>
+            <format>R8G8B8</format>
+        </image>
+        <clip>
+            <near>0.02</near>
+            <far>300</far>
+        </clip>
+        <noise>
+            <type>gaussian</type>
+            <mean>0.0</mean>
+            <stddev>0.001</stddev>
+        </noise>
+        <distortion>
+          <k1>-0.264598808</k1>
+          <k2>0.0156281135</k2>
+          <k3>0.0822019378</k3>
+          <p1>0.0000652954</p1>
+          <p2>0.0053984313</p2>
+        </distortion>
+        <optical_frame_id>camera_csi_front_optical_link</optical_frame_id>
+        <camera_info_topic>qcar/csi_front/camera_info</camera_info_topic>
+      </camera>
+    </sensor>
+  </gazebo>
+  <link name="camera_csi_right_optical_link"/>
+  <joint name="camera_csi_right_optical_joint" type="fixed">
+    <!-- these values have to be these values otherwise the gazebo camera
+        image won't be aligned properly with the frame it is supposedly
+        originating from -->
+    <origin xyz="0 0 0" rpy="${-pi/2} 0 ${-pi/2}"/>
+    <parent link="camera_csi_right"/>
+    <child link="camera_csi_right_optical_link"/>
+  </joint>
+<!-- Define all the computer vision sernsor properties -->
+	<gazebo reference="camera_csi_right">
+    <!-- <material>Gazebo/Green</material> -->
+    <sensor type="camera" name="csi_right">
+      <always_on>1</always_on>
+      <update_rate>60.0</update_rate>
+      <visualize>true</visualize>
+      <topic>qcar/csi_right/image_raw</topic>
+      <camera name="right">
+        <horizontal_fov>2.79253</horizontal_fov>
+        <image>
+            <width>1280</width>
+            <height>640</height>
+            <format>R8G8B8</format>
+        </image>
+        <clip>
+            <near>0.02</near>
+            <far>300</far>
+        </clip>
+        <noise>
+            <type>gaussian</type>
+            <mean>0.0</mean>
+            <stddev>0.001</stddev>
+        </noise>
+        <distortion>
+          <k1>-0.264598808</k1>
+          <k2>0.0156281135</k2>
+          <k3>0.0822019378</k3>
+          <p1>0.0000652954</p1>
+          <p2>0.0053984313</p2>
+        </distortion>
+        <optical_frame_id>camera_csi_right_optical_link</optical_frame_id>
+        <camera_info_topic>qcar/csi_right/camera_info</camera_info_topic>
+      </camera>
+    </sensor>
+  </gazebo>
+  <link name="camera_csi_left_optical_link"/>
+  <joint name="camera_csi_left_optical_joint" type="fixed">
+    <!-- these values have to be these values otherwise the gazebo camera
+        image won't be aligned properly with the frame it is supposedly
+        originating from -->
+    <origin xyz="0 0 0" rpy="${-pi/2} 0 ${-pi/2}"/>
+    <parent link="camera_csi_left"/>
+    <child link="camera_csi_left_optical_link"/>
+  </joint>
+<!-- Define all the computer vision sernsor properties -->
+	<gazebo reference="camera_csi_left">
+    <!-- <material>Gazebo/Green</material> -->
+    <sensor type="camera" name="csi_left">
+      <always_on>1</always_on>
+      <update_rate>60.0</update_rate>
+      <visualize>true</visualize>
+      <topic>qcar/csi_left/image_raw</topic>
+      <camera name="front">
+        <horizontal_fov>2.79253</horizontal_fov>
+        <image>
+            <width>1280</width>
+            <height>640</height>
+            <format>R8G8B8</format>
+        </image>
+        <clip>
+            <near>0.02</near>
+            <far>300</far>
+        </clip>
+        <noise>
+            <type>gaussian</type>
+            <mean>0.0</mean>
+            <stddev>0.001</stddev>
+        </noise>
+        <distortion>
+          <k1>-0.264598808</k1>
+          <k2>0.0156281135</k2>
+          <k3>0.0822019378</k3>
+          <p1>0.0000652954</p1>
+          <p2>0.0053984313</p2>
+        </distortion>
+        <optical_frame_id>camera_csi_left_optical_link</optical_frame_id>
+        <camera_info_topic>qcar/csi_left/camera_info</camera_info_topic>
+      </camera>
+    </sensor>
+  </gazebo>
+  <link name="camera_csi_back_optical_link"/>
+  <joint name="camera_csi_back_optical_joint" type="fixed">
+    <!-- these values have to be these values otherwise the gazebo camera
+        image won't be aligned properly with the frame it is supposedly
+        originating from -->
+    <origin xyz="0 0 0" rpy="${-pi/2} 0 ${-pi/2}"/>
+    <parent link="camera_csi_back"/>
+    <child link="camera_csi_back_optical_link"/>
+  </joint>
+<!-- Define all the computer vision sernsor properties -->
+	<gazebo reference="camera_csi_back">
+    <!-- <material>Gazebo/Green</material> -->
+    <sensor type="camera" name="csi_back">
+      <always_on>1</always_on>
+      <update_rate>60.0</update_rate>
+      <visualize>true</visualize>
+      <topic>qcar/csi_back/image_raw</topic>
+      <camera name="front">
+        <horizontal_fov>2.79253</horizontal_fov>
+        <image>
+            <width>1280</width>
+            <height>640</height>
+            <format>R8G8B8</format>
+        </image>
+        <clip>
+            <near>0.02</near>
+            <far>300</far>
+        </clip>
+        <noise>
+            <type>gaussian</type>
+            <mean>0.0</mean>
+            <stddev>0.001</stddev>
+        </noise>
+        <distortion>
+          <k1>-0.264598808</k1>
+          <k2>0.0156281135</k2>
+          <k3>0.0822019378</k3>
+          <p1>0.0000652954</p1>
+          <p2>0.0053984313</p2>
+        </distortion>
+        <optical_frame_id>camera_csi_back_optical_link</optical_frame_id>
+        <camera_info_topic>qcar/csi_back/camera_info</camera_info_topic>
+      </camera>
+    </sensor>
+  </gazebo>
+  <!-- Gazebo Parameters -->
+    <gazebo reference="base">
+      <mu1>0.0001</mu1>
+      <mu2>0.0001</mu2>
+    </gazebo>
+    <gazebo reference="right_front_wheel">
+      <mu1>100.0</mu1>
+      <mu2>100.0</mu2>
+    </gazebo>
+    <gazebo reference="left_front_wheel">
+      <mu1>100.0</mu1>
+      <mu2>100.0</mu2>
+    </gazebo>
+    <gazebo reference="right_rear_wheel">
+      <mu1>100.0</mu1>
+      <mu2>100.0</mu2>
+    </gazebo>
+    <gazebo reference="left_rear_wheel">
+      <mu1>100.0</mu1>
+      <mu2>100.0</mu2>
+    </gazebo>
   <!-- Gazebo Control -->
   <ros2_control name="control" type="system">

File: qcar_description/urdf/qcar_ros2.urdf.xacro (robot description, xacro)
@@ -502,25 +502,4 @@
     </joint>
     <!-- The above is for the wheels and turning etc -->
-    <!-- Gazebo Parameters -->
-    <gazebo reference="base">
-      <mu1>0.0001</mu1>
-      <mu2>0.0001</mu2>
-    </gazebo>
-    <gazebo reference="right_front_wheel">
-      <mu1>100.0</mu1>
-      <mu2>100.0</mu2>
-    </gazebo>
-    <gazebo reference="left_front_wheel">
-      <mu1>100.0</mu1>
-      <mu2>100.0</mu2>
-    </gazebo>
-    <gazebo reference="right_rear_wheel">
-      <mu1>100.0</mu1>
-      <mu2>100.0</mu2>
-    </gazebo>
-    <gazebo reference="left_rear_wheel">
-      <mu1>100.0</mu1>
-      <mu2>100.0</mu2>
-    </gazebo>
     <!--<gazebo>
       <plugin name="gazebo_ros_control" filename="libgazebo_ros_control.so" />

File: qcar_description/urdf/qcar_system.urdf.xacro (robot description, xacro)
@@ -9,13 +9,4 @@
   <!-- Import all Gazebo-customization elements, including Gazebo colors -->
   <xacro:include filename="$(find qcar_description)/urdf/qcar.gazebo.xacro" />
-  <!-- Import Rviz colors -->
-  <!-- <xacro:include filename="$(find qcar_description)/urdf/qcar.materials.xacro" /> -->
-  <!-- Import diffbot ros2_control description -->
-  <!-- <xacro:include filename="$(find qcar_description)/ros2_control/qcar_system.ros2_control.xacro" /> -->
-  <!-- Used for fixing robot -->
-  <!-- <link name="world"/> -->
-  <!-- <gazebo reference="world">
-    <static>false</static>
-  </gazebo> -->
   <xacro:QCar parent="world" prefix="$(arg prefix)">
     <origin xyz="0 0 0" rpy="0 0 0" />
