Commit message: added: imu sensor to qcar and adapted odom to work with nav2
Co-authored-by: Copilot <copilot@github.com>

File: qcar_description/urdf/qcar.gazebo.xacro (robot description, xacro)
@@ -286,8 +286,58 @@
         <visualize>true</visualize>
         <topic>imu</topic>
+        <gz_frame_id>imu</gz_frame_id>
         <imu>
-          <orientation_reference_frame>
-            <localization>GRAV_UP</localization>
-          </orientation_reference_frame>
+          <angular_velocity>
+            <x>
+              <noise type="gaussian">
+                <mean>0.0</mean>
+                <stddev>2e-4</stddev>
+                <bias_mean>0.0000075</bias_mean>
+                <bias_stddev>0.0000008</bias_stddev>
+              </noise>
+            </x>
+            <y>
+              <noise type="gaussian">
+                <mean>0.0</mean>
+                <stddev>2e-4</stddev>
+                <bias_mean>0.0000075</bias_mean>
+                <bias_stddev>0.0000008</bias_stddev>
+              </noise>
+            </y>
+            <z>
+              <noise type="gaussian">
+                <mean>0.0</mean>
+                <stddev>2e-4</stddev>
+                <bias_mean>0.0000075</bias_mean>
+                <bias_stddev>0.0000008</bias_stddev>
+              </noise>
+            </z>
+          </angular_velocity>
+          <linear_acceleration>
+            <x>
+              <noise type="gaussian">
+                <mean>0.0</mean>
+                <stddev>1.7e-2</stddev>
+                <bias_mean>0.1</bias_mean>
+                <bias_stddev>0.001</bias_stddev>
+              </noise>
+            </x>
+            <y>
+              <noise type="gaussian">
+                <mean>0.0</mean>
+                <stddev>1.7e-2</stddev>
+                <bias_mean>0.1</bias_mean>
+                <bias_stddev>0.001</bias_stddev>
+              </noise>
+            </y>
+            <z>
+              <noise type="gaussian">
+                <mean>0.0</mean>
+                <stddev>1.7e-2</stddev>
+                <bias_mean>0.1</bias_mean>
+                <bias_stddev>0.001</bias_stddev>
+              </noise>
+            </z>
+          </linear_acceleration>
         </imu>
       <!-- Sensor |camera,ray,imu,magnetometer,gps,force_torque,contact,sonar,rfidtag,rfid| -->
@@ -312,6 +362,8 @@
         </plugin>
         <plugin filename="gz-sim-odometry-publisher-system" name="gz::sim::systems::OdometryPublisher">
-          <odom_frame>vehicle/odom</odom_frame>
-          <robot_base_frame>base_link</robot_base_frame>
+          <odom_frame>odom</odom_frame>
+          <robot_base_frame>base_footprint</robot_base_frame>
+        </plugin>
+        <plugin filename="gz-sim-imu-system" name="gz::sim::systems::Imu">
         </plugin>
       </xacro:unless>
@@ -332,7 +384,9 @@
             <render_engine>ogre2</render_engine>
         </plugin>
-        <plugin filename="ignition-gazebo-odometry-publisher-system" name="ignition::gazebo::systems::OdometryPublisher">
-          <odom_frame>vehicle/odom</odom_frame>
-          <robot_base_frame>base_link</robot_base_frame>
+        <plugin filename="libignition-gazebo-odometry-publisher-system" name="ignition::gazebo::systems::OdometryPublisher">
+          <odom_frame>odom</odom_frame>
+          <robot_base_frame>base_footprint</robot_base_frame>
+        </plugin>
+        <plugin filename="libignition-gazebo-imu-system" name="ignition::gazebo::systems::Imu">
         </plugin>
       </xacro:if>

File: qcar_description/urdf/qcar_ros2.urdf.xacro (robot description, xacro)
@@ -123,14 +123,14 @@
       </inertial>
     </xacro:macro>
-    <!-- base_link must have geometry so that its axes can be displayed in
+    <!-- base_footprint must have geometry so that its axes can be displayed in
          rviz. -->
     <!-- <joint name="$base_joint" type="fixed">
       <xacro:insert_block name="origin" />
       <parent link="${parent}"/>
-      <child link="${prefix}base_link" />
+      <child link="${prefix}base_footprint" />
     </joint> -->
-   <link name="base_link" />
+   <link name="base_footprint" />
     <!-- Chassis -->
-    <link name="base">
+    <link name="base_link">
       <visual>
         <!-- <origin xyz="0 0 ${-chassis_height / 2}"/> -->
@@ -167,10 +167,10 @@
     </link>
   <!-- ________below is all about lidar positions and camera positions______________ -->
-    <joint name="base_link_to_chasis" type="fixed">
-      <parent link="base_link"/>
-      <child link="base"/>
+    <joint name="base_footprint_to_chasis" type="fixed">
+      <parent link="base_footprint"/>
+      <child link="base_link"/>
     </joint>
     <joint name="body_lidar_joint" type="fixed">
-    <parent link="base"/>
+    <parent link="base_link"/>
     <child link="lidar"/>
     <origin rpy="0 0 0" xyz="-0.01227 -0.00045 0.16152"/>
@@ -203,5 +203,5 @@
         <origin rpy="0 0 0" xyz="0.081686 0.031547 0.15445"/>
         <!-- <origin rpy="0 0 0" xyz="0 0 0"/> -->
-      <parent link="base"/>
+      <parent link="base_link"/>
       <child link="camera_rgb"/>
     </joint>
@@ -212,5 +212,5 @@
         <origin rpy="0 0 0" xyz="0.19236 -0.000475 0.093029"/>
         <!-- <origin rpy="0 0 0" xyz="0 0 0"/> -->
-        <parent link="base"/>
+        <parent link="base_link"/>
         <child link="camera_csi_front"/>
     </joint>
@@ -223,5 +223,5 @@
         <origin rpy="0 0 -1.5708" xyz="0.012887 -0.06755 0.093029"/>
         <!-- <origin rpy="0 0 0" xyz="0 0 0"/> -->
-        <parent link="base"/>
+        <parent link="base_link"/>
         <child link="camera_csi_right"/>
     </joint>
@@ -232,5 +232,5 @@
         <origin rpy="0 0 -3.1416" xyz="-0.16669 -0.000578 0.093029"/>
         <!-- <origin rpy="0 0 0" xyz="0 0 0"/> -->
-        <parent link="base"/>
+        <parent link="base_link"/>
         <child link="camera_csi_back"/>
     </joint>
@@ -243,5 +243,5 @@
          <origin rpy="0 0 1.5708" xyz="0.012784 0.052497 0.093029"/>
         <!-- <origin rpy="0 0 0" xyz="0 0 0"/> -->
-        <parent link="base"/>
+        <parent link="base_link"/>
         <child link="camera_csi_left"/>
     </joint>
@@ -254,5 +254,5 @@
          <origin rpy="0 0 0" xyz="0.1278 0.0223 0.087229"/>
         <!-- <origin rpy="0 0 0" xyz="0 0 0"/> -->
-        <parent link="base"/>
+        <parent link="base_link"/>
         <child link="imu"/>
     </joint>
@@ -267,8 +267,8 @@
         </actuator>
     </transmission> -->
-    <!-- ___base_link - > left_front_position_joint (fixed) -> left_steering_link -> left_steering_joint(revolote) -> left_front_axle_carrier -> left_front_axle(joint) (continuous) -> left_front_wheel_______________ -->
+    <!-- ___base_footprint - > left_front_position_joint (fixed) -> left_steering_link -> left_steering_joint(revolote) -> left_front_axle_carrier -> left_front_axle(joint) (continuous) -> left_front_wheel_______________ -->
     <!-- The "wheel" macro defines an axle carrier, axle, and wheel. -->
     <joint name="left_front_position_joint" type="fixed">
-      <parent link="base"/>
+      <parent link="base_link"/>
       <child link="left_steering_link"/>
       <origin rpy="0 0 0" xyz="0.12960 0.05590 0.03338"/>
@@ -348,5 +348,5 @@
       </actuator>
     </transmission>
-  <!-- ___base_link - > right_front_position_joint (fixed) -> right_steering_link -> right_steering_joint(revolote) -> right_front_axle_carrier -> right_front_axle(joint) (continuous) -> right_front_wheel_______________ -->
+  <!-- ___base_footprint - > right_front_position_joint (fixed) -> right_steering_link -> right_steering_joint(revolote) -> right_front_axle_carrier -> right_front_axle(joint) (continuous) -> right_front_wheel_______________ -->
     <link name="right_front_axle_carrier">
       <xacro:null_inertial/>
@@ -391,5 +391,5 @@
     </link>
     <joint name="right_front_position_joint" type="fixed">
-      <parent link="base"/>
+      <parent link="base_link"/>
       <child link="right_steering_link"/>
       <origin rpy="0 0 0" xyz="0.12960 -0.05590 0.03338"/>
@@ -430,5 +430,5 @@
     <!-- The upper portion is for the front -->
     <!-- Now is for the rear which only has axles -->
-  <!-- ____base_link -> left_rear_position_joint(fixed) -> left_rear_axle_carrier -> left_rear_axle (joint)(continuous) -> left_rear_wheel_____ -->
+  <!-- ____base_footprint -> left_rear_position_joint(fixed) -> left_rear_axle_carrier -> left_rear_axle (joint)(continuous) -> left_rear_wheel_____ -->
     <link name="left_rear_axle_carrier">
       <xacro:null_inertial/>
@@ -472,9 +472,9 @@
     </link>
     <joint name="left_rear_position_joint" type="fixed">
-      <parent link="base"/>
+      <parent link="base_link"/>
       <child link="left_rear_axle_carrier"/>
       <origin rpy="0 0 0" xyz="-0.12765 0.05610 0.03338"/>
     </joint>
-  <!-- ____base_link -> right_rear_position_joint(fixed) -> right_rear_axle_carrier -> right_rear_axle (joint)(continuous) -> right_rear_wheel_____ -->
+  <!-- ____base_footprint -> right_rear_position_joint(fixed) -> right_rear_axle_carrier -> right_rear_axle (joint)(continuous) -> right_rear_wheel_____ -->
     <link name="right_rear_axle_carrier">
       <xacro:null_inertial/>
@@ -517,5 +517,5 @@
     </link>
     <joint name="right_rear_position_joint" type="fixed">
-      <parent link="base"/>
+      <parent link="base_link"/>
       <child link="right_rear_axle_carrier"/>
       <origin rpy="0 0 0" xyz="-0.12765 -0.05610 0.03338"/>
@@ -523,5 +523,5 @@
     <!-- The above is for the wheels and turning etc -->
     <!-- Gazebo Parameters -->
-    <gazebo reference="base">
+    <gazebo reference="base_link">
       <mu1>0.0001</mu1>
       <mu2>0.0001</mu2>
@@ -613,5 +613,5 @@
       <plugin name="gazebo_ros_p3d"     filename="libgazebo_ros_p3d.so">
         <frameName>map</frameName>
-        <bodyName>base_link</bodyName>
+        <bodyName>base_footprint</bodyName>
         <topicName>odom_truth</topicName>
         <updateRate>30.0</updateRate>
