Commit message: solved conflicts

File: ackermann_vehicle_description/urdf/ackermann_robot.urdf.xacro (robot description, xacro)
@@ -3,5 +3,6 @@
     <xacro:include filename="$(find ackermann_vehicle_description)/urdf/mobile_base.xacro" />
     <xacro:arg name="robot_parameters_file" default="$(find ackermann_vehicle_description)/config/params.yaml"/>
-    <xacro:ackermann_robot robot_parameters_file="${robot_parameters_file}">
-    </xacro:ackermann_robot>
+    <xacro:ackermann_robot
+        robot_parameters_file="${robot_parameters_file}"
+    />
 </robot>

File: ackermann_vehicle_description/urdf/common_properties.xacro (robot description, xacro)
@@ -45,20 +45,20 @@
         <xacro:property name="steering_parameters" value="${parameters['robot_parameters']['steering']}" />
         <!-- Parameters for the base -->
-        <xacro:property name="base_length" value="${base_parameters[base_length]}" scope="parent"/>
-        <xacro:property name="base_width" value="${base_parameters[base_width]}" scope="parent"/>
-        <xacro:property name="base_height" value="${base_parameters[base_height]}" scope="parent"/>
-        <xacro:property name="base_density" value="${base_parameters[base_density]}" scope="parent"/>
+        <xacro:property name="base_length" value="${base_parameters['base_length']}" scope="parent"/>
+        <xacro:property name="base_width" value="${base_parameters['base_width']}" scope="parent"/>
+        <xacro:property name="base_height" value="${base_parameters['base_height']}" scope="parent"/>
+        <xacro:property name="base_density" value="${base_parameters['base_density']}" scope="parent"/>
         <!-- Parameters for the wheels -->
-        <xacro:property name="wheel_radius" value="${wheel_parameters[wheel_radius]}" scope="parent"/>
-        <xacro:property name="wheel_width" value="${wheel_parameters[wheel_width]}" scope="parent"/>
-        <xacro:property name="wheel_density" value="${wheel_parameters[wheel_density]}" scope="parent"/>
+        <xacro:property name="wheel_radius" value="${wheel_parameters['wheel_radius']}" scope="parent"/>
+        <xacro:property name="wheel_width" value="${wheel_parameters['wheel_width']}" scope="parent"/>
+        <xacro:property name="wheel_density" value="${wheel_parameters['wheel_density']}" scope="parent"/>
         <!-- Parameters for the steering -->
-        <xacro:property name="max_steering_angle" value="${steering_parameters[max_steering_angle]}" scope="parent"/>
-        <xacro:property name="max_steering_angular_velocity" value="${steering_parameters[max_steering_angular_velocity]}" scope="parent"/>
-        <xacro:property name="max_velocity" value="${steering_parameters[max_velocity]}" scope="parent"/>
-        <xacro:property name="max_effort" value="${steering_parameters[max_effort]}" scope="parent"/>
-        <xacro:property name="max_steering_effort" value="${steering_parameters[max_steering_effort]}" scope="parent"/>
+        <xacro:property name="max_steering_angle" value="${steering_parameters['max_steering_angle']}" scope="parent"/>
+        <xacro:property name="max_steering_angular_velocity" value="${steering_parameters['max_steering_angular_velocity']}" scope="parent"/>
+        <xacro:property name="max_velocity" value="${steering_parameters['max_velocity']}" scope="parent"/>
+        <xacro:property name="max_effort" value="${steering_parameters['max_effort']}" scope="parent"/>
+        <xacro:property name="max_steering_effort" value="${steering_parameters['max_steering_effort']}" scope="parent"/>
         <xacro:property name="base_mass" value="${base_density * base_length * base_height * base_width}" scope="parent"/>
-        <xacro:property name="wheel_separation" value="${base_width + wheel_width}" scope="global"/>
+        <xacro:property name="wheel_separation" value="${base_width + wheel_width}" scope="parent"/>
         <xacro:property name="wheel_offset" value="${base_length/2 - wheel_radius}" scope="parent"/>
         <xacro:property name="wheel_mass" value="${wheel_density * pi * wheel_radius * wheel_radius * wheel_width}" scope="parent"/>

Commit message: Created and tested the display launch

File: ackermann_vehicle_description/urdf/ackermann_robot.urdf.xacro (robot description, xacro)
@@ -4,5 +4,5 @@
     <xacro:arg name="robot_parameters_file" default="$(find ackermann_vehicle_description)/config/params.yaml"/>
     <xacro:ackermann_robot
-        robot_parameters_file="${robot_parameters_file}"
+        robot_parameters_file="$(arg robot_parameters_file)"
     />
 </robot>

File: ackermann_vehicle_description/urdf/mobile_base.xacro (robot description, xacro)
@@ -40,4 +40,23 @@
             </collision>
         </link>
+        <xacro:wheel_link prefix="rear_right"/>
+        <xacro:wheel_link prefix="rear_left"/>
+        <joint name="base_joint" type="fixed">
+            <parent link="base_footprint"/>
+            <child link="base_link"/>
+            <origin xyz="0.0 0.0 ${wheel_radius}" rpy="0.0 0.0 0.0"/>
+        </joint>
+        <joint name="rear_right_wheel_joint" type="continuous">
+            <parent link="base_link"/>
+            <child link="rear_right_wheel_link"/>
+            <axis xyz="0 1 0"/>
+            <origin xyz="${-wheel_offset} ${-wheel_separation/2} 0" rpy="0 0 0"/>
+        </joint>
+        <joint name="rear_left_wheel_joint" type="continuous">
+            <parent link="base_link"/>
+            <child link="rear_left_wheel_link"/>
+            <axis xyz="0 1 0"/>
+            <origin xyz="${-wheel_offset} ${wheel_separation/2} 0" rpy="0 0 0"/>
+        </joint>
     </xacro:macro>
 </robot>

Commit message: Finalizados los paquetes del vehiculo Ackermann

File: ackermann_vehicle_description/urdf/ackermann_robot.urdf.xacro (robot description, xacro)
@@ -6,3 +6,4 @@
         robot_parameters_file="$(arg robot_parameters_file)"
     />
+    <xacro:include filename="$(find ackermann_vehicle_description)/urdf/mobile_base_gazebo.xacro" />
 </robot>

File: ackermann_vehicle_description/urdf/common_properties.xacro (robot description, xacro)
@@ -50,16 +50,16 @@
         <xacro:property name="base_density" value="${base_parameters['base_density']}" scope="parent"/>
         <!-- Parameters for the wheels -->
-        <xacro:property name="wheel_radius" value="${wheel_parameters['wheel_radius']}" scope="parent"/>
+        <xacro:property name="wheel_radius" value="${wheel_parameters['wheel_radius']}" scope="global"/>
         <xacro:property name="wheel_width" value="${wheel_parameters['wheel_width']}" scope="parent"/>
         <xacro:property name="wheel_density" value="${wheel_parameters['wheel_density']}" scope="parent"/>
         <!-- Parameters for the steering -->
-        <xacro:property name="max_steering_angle" value="${steering_parameters['max_steering_angle']}" scope="parent"/>
+        <xacro:property name="max_steering_angle" value="${steering_parameters['max_steering_angle']}" scope="global"/>
         <xacro:property name="max_steering_angular_velocity" value="${steering_parameters['max_steering_angular_velocity']}" scope="parent"/>
-        <xacro:property name="max_velocity" value="${steering_parameters['max_velocity']}" scope="parent"/>
+        <xacro:property name="max_velocity" value="${steering_parameters['max_velocity']}" scope="global"/>
         <xacro:property name="max_effort" value="${steering_parameters['max_effort']}" scope="parent"/>
         <xacro:property name="max_steering_effort" value="${steering_parameters['max_steering_effort']}" scope="parent"/>
         <xacro:property name="base_mass" value="${base_density * base_length * base_height * base_width}" scope="parent"/>
-        <xacro:property name="wheel_separation" value="${base_width + wheel_width}" scope="parent"/>
-        <xacro:property name="wheel_offset" value="${base_length/2 - wheel_radius}" scope="parent"/>
+        <xacro:property name="wheel_separation" value="${base_width + wheel_width}" scope="global"/>
+        <xacro:property name="wheel_offset" value="${base_length/2 - wheel_radius}" scope="global"/>
         <xacro:property name="wheel_mass" value="${wheel_density * pi * wheel_radius * wheel_radius * wheel_width}" scope="parent"/>
         <xacro:property name="max_wheel_angular_velocity" value="${max_velocity / wheel_radius}" scope="parent"/>

File: ackermann_vehicle_description/urdf/mobile_base.xacro (robot description, xacro)
@@ -18,4 +18,22 @@
                 </geometry>
                 <origin xyz="0 0 0" rpy="${pi/2} 0 0" />
+            </collision>
+        </link>
+    </xacro:macro>
+    <xacro:macro name="steering_link" params="prefix">
+        <link name="${prefix}_steering_link">
+            <xacro:cylinder_inertia r="0.01" l="0.001" m="0.01" o_xyz="0.0 0.0 0.0" o_rpy="${pi / 2.0} 0.0 0.0"/>
+            <visual>
+                <origin xyz="0.0 0.0 0.0" rpy="${pi / 2.0} 0.0 0.0"/>
+                <geometry>
+                    <cylinder length="0.001" radius="0.01"/>
+                </geometry>
+                <material name="black"/>
+                </visual>
+            <collision>
+                <origin xyz="0.0 0.0 0.0" rpy="${pi / 2.0} 0.0 0.0"/>
+                <geometry>
+                    <cylinder length="0.001" radius="0.01"/>
+                </geometry>
             </collision>
         </link>
@@ -42,4 +60,8 @@
         <xacro:wheel_link prefix="rear_right"/>
         <xacro:wheel_link prefix="rear_left"/>
+        <xacro:steering_link prefix="front_right"/>
+        <xacro:steering_link prefix="front_left"/>
+        <xacro:wheel_link prefix="front_right"/>
+        <xacro:wheel_link prefix="front_left"/>
         <joint name="base_joint" type="fixed">
             <parent link="base_footprint"/>
@@ -50,12 +72,48 @@
             <parent link="base_link"/>
             <child link="rear_right_wheel_link"/>
+            <origin xyz="-${wheel_offset} ${-wheel_separation/2} 0.0" rpy="0.0 0.0 0.0"/>
             <axis xyz="0 1 0"/>
-            <origin xyz="${-wheel_offset} ${-wheel_separation/2} 0" rpy="0 0 0"/>
+            <limit effort="${max_effort}" velocity="${max_wheel_angular_velocity}"/>
+            <dynamics damping="0.1" friction="0.1"/>
         </joint>
         <joint name="rear_left_wheel_joint" type="continuous">
             <parent link="base_link"/>
             <child link="rear_left_wheel_link"/>
+            <origin xyz="-${wheel_offset} ${wheel_separation/2} 0.0" rpy="0.0 0.0 0.0"/>
             <axis xyz="0 1 0"/>
-            <origin xyz="${-wheel_offset} ${wheel_separation/2} 0" rpy="0 0 0"/>
+            <limit effort="${max_effort}" velocity="${max_wheel_angular_velocity}"/>
+            <dynamics damping="0.1" friction="0.1"/>
+        </joint>
+        <joint name="front_right_steering_joint" type="revolute">
+            <parent link="base_link"/>
+            <child link="front_right_steering_link"/>
+            <origin xyz="${wheel_offset} ${-wheel_separation/2} 0.0" rpy="0.0 0.0 0.0"/>
+            <axis xyz="0 0 1"/>
+            <limit effort="${max_steering_effort}" lower="${-max_steering_angle}" upper="${max_steering_angle}" velocity="${max_steering_angular_velocity}"/>
+            <dynamics damping="0.1" friction="0.1"/>
+        </joint>
+        <joint name="front_right_wheel_joint" type="continuous">
+            <parent link="front_right_steering_link"/>
+            <child link="front_right_wheel_link"/>
+            <origin xyz="0.0 0.0 0.0" rpy="0.0 0.0 0.0"/>
+            <axis xyz="0 1 0"/>
+            <limit effort="${max_effort}" velocity="${max_wheel_angular_velocity}"/>
+            <dynamics damping="0.1" friction="0.1"/>
+        </joint>
+        <joint name="front_left_steering_joint" type="revolute">
+            <parent link="base_link"/>
+            <child link="front_left_steering_link"/>
+            <origin xyz="${wheel_offset} ${wheel_separation/2} 0.0" rpy="0.0 0.0 0.0"/>
+            <axis xyz="0 0 1"/>
+            <limit effort="${max_steering_effort}" lower="${-max_steering_angle}" upper="${max_steering_angle}" velocity="${max_steering_angular_velocity}"/>
+            <dynamics damping="0.1" friction="0.1"/>
+        </joint>
+        <joint name="front_left_wheel_joint" type="continuous">
+            <parent link="front_left_steering_link"/>
+            <child link="front_left_wheel_link"/>
+            <origin xyz="0.0 0.0 0.0" rpy="0.0 0.0 0.0"/>
+            <axis xyz="0 1 0"/>
+            <limit effort="${max_effort}" velocity="${max_wheel_angular_velocity}"/>
+            <dynamics damping="0.1" friction="0.1"/>
         </joint>
     </xacro:macro>

Commit message: test: nav in ackermann

File: ackermann_vehicle_description/urdf/ackermann_robot.urdf.xacro (robot description, xacro)
@@ -7,3 +7,4 @@
     />
     <xacro:include filename="$(find ackermann_vehicle_description)/urdf/mobile_base_gazebo.xacro" />
+    <xacro:include filename="$(find ackermann_vehicle_description)/urdf/lidar.xacro"/>
 </robot>

File: ackermann_vehicle_description/urdf/common_properties.xacro (robot description, xacro)
@@ -47,5 +47,5 @@
         <xacro:property name="base_length" value="${base_parameters['base_length']}" scope="parent"/>
         <xacro:property name="base_width" value="${base_parameters['base_width']}" scope="parent"/>
-        <xacro:property name="base_height" value="${base_parameters['base_height']}" scope="parent"/>
+        <xacro:property name="base_height" value="${base_parameters['base_height']}" scope="global"/>
         <xacro:property name="base_density" value="${base_parameters['base_density']}" scope="parent"/>
         <!-- Parameters for the wheels -->
